Commit message: first working nav2

File: husky_description/urdf/husky_macro.urdf.xacro (robot description, xacro)
@@ -73,4 +73,16 @@
       <parent link="${prefix}base_link" />
       <child link="${prefix}inertial_link" />
+    </joint>
+    <link name="${prefix}velodyne">
+      <inertial>
+        <mass value="46.034" />
+        <origin xyz="-0.00065 -0.085 0.062" />
+        <inertia ixx="0.6022" ixy="-0.02364" ixz="-0.1197" iyy="1.7386" iyz="-0.001544" izz="2.0296" />
+      </inertial>
+    </link>
+    <joint name="${prefix}velodyne_joint" type="fixed">
+      <origin xyz="0 0 0" rpy="0 0 0" />
+      <parent link="${prefix}base_link" />
+      <child link="${prefix}velodyne" />
     </joint>
     <!-- IMU Link-->
